File: doc/schematic/schematic.kicad_sch (KiCad schematic)
At the start: 11 parts, among them J1 Conn_01x06_Pin, J10 HAND1, J15 AV7V, J2 AC9V*2, J3 MOTOR, J4 AC24V, J5 Conn_01x06_Pin, J6 TRANS, J7 AC, J8 HAND2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

Commit message: Added ST862D-P2_schematic.pdf
Other:
- company: (none) -> 4Source
Changed lines of the file:
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@@
   (title_block
     (title "ST-862D-P2")
+    (date "2023-06-10")
+    (company "4Source")
   )
   (no_connect (at 113.03 53.34))
