File: doc/schematic/ST862D-P2/schematic.kicad_sch (KiCad schematic)
At the start: 11 parts, among them J1 Conn_01x06_Pin, J10 HAND1, J15 AV7V, J2 AC9V*2, J3 MOTOR, J4 AC24V, J5 Conn_01x06_Pin, J6 TRANS, J7 AC, J8 HAND2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

Commit message: Update Schematics
Parts:
- added S1, S2: 1, symbol Switch:SW_Push
- added S3: 3, symbol Switch:SW_Push
- added S4: AIR_DOWN, symbol Switch:SW_Push
- added S5: AIR_UP, symbol Switch:SW_Push
- added S6: TEMP_DOWN, symbol Switch:SW_Push
- added S7: TEMP_UP, symbol Switch:SW_Push
- renumbered J8 to J9
Connections:
- net GND: now also S1.1, S2.1, S3.1, S4.1, S5.1, S6.1, S7.1
